Commit message: camera

File: urdf/AutoCar.xacro (robot description, xacro)
@@ -6,7 +6,7 @@
 <link name="base_link">
   <inertial>
-    <origin xyz="-0.003146316924459841 -1.0874806484475148e-16 0.032267635209005975" rpy="0 0 0"/>
-    <mass value="42.01731210785512"/>
-    <inertia ixx="0.137212" iyy="1.462636" izz="1.568445" ixy="-0.0" iyz="-0.0" ixz="-0.000365"/>
+    <origin xyz="-0.0008559347867336729 -1.0776657557532648e-16 0.032797715315650726" rpy="0 0 0"/>
+    <mass value="42.39998679844243"/>
+    <inertia ixx="0.138613" iyy="1.488522" izz="1.592956" ixy="-0.0" iyz="-0.0" ixz="-0.006017"/>
   </inertial>
   <visual>
@@ -101,4 +101,44 @@
     <geometry>
       <mesh filename="file://$(find auto_car_description)/meshes/rear_right_wheel_1.stl" scale="0.001 0.001 0.001"/>
+    </geometry>
+  </collision>
+</link>
+<link name="camera_rotate_servo_1">
+  <inertial>
+    <origin xyz="0.001018906391389518 -1.7763568394002506e-16 0.00999999999998398" rpy="0 0 0"/>
+    <mass value="0.3675302288901849"/>
+    <inertia ixx="9e-05" iyy="8.9e-05" izz="0.000152" ixy="0.0" iyz="0.0" ixz="-0.0"/>
+  </inertial>
+  <visual>
+    <origin xyz="-0.250626 -0.0 -0.116" rpy="0 0 0"/>
+    <geometry>
+      <mesh filename="file://$(find auto_car_description)/meshes/camera_rotate_servo_1.stl" scale="0.001 0.001 0.001"/>
+    </geometry>
+    <material name="silver"/>
+  </visual>
+  <collision>
+    <origin xyz="-0.250626 -0.0 -0.116" rpy="0 0 0"/>
+    <geometry>
+      <mesh filename="file://$(find auto_car_description)/meshes/camera_rotate_servo_1.stl" scale="0.001 0.001 0.001"/>
+    </geometry>
+  </collision>
+</link>
+<link name="camera_tilt_servo_1">
+  <inertial>
+    <origin xyz="0.02297270847794408 3.293785511004899e-10 1.1765838303645637e-11" rpy="0 0 0"/>
+    <mass value="0.09526148376679884"/>
+    <inertia ixx="5.4e-05" iyy="5.3e-05" izz="0.000103" ixy="-0.0" iyz="-0.0" ixz="-0.0"/>
+  </inertial>
+  <visual>
+    <origin xyz="-0.235626 -0.0 -0.126" rpy="0 0 0"/>
+    <geometry>
+      <mesh filename="file://$(find auto_car_description)/meshes/camera_tilt_servo_1.stl" scale="0.001 0.001 0.001"/>
+    </geometry>
+    <material name="silver"/>
+  </visual>
+  <collision>
+    <origin xyz="-0.235626 -0.0 -0.126" rpy="0 0 0"/>
+    <geometry>
+      <mesh filename="file://$(find auto_car_description)/meshes/camera_tilt_servo_1.stl" scale="0.001 0.001 0.001"/>
     </geometry>
   </collision>
@@ -158,3 +198,15 @@
   <axis xyz="0.0 -1.0 0.0"/>
 </joint>
+<joint name="joint_cam_rotate" type="continuous">
+  <origin xyz="0.250626 0.0 0.116" rpy="0 0 0"/>
+  <parent link="base_link"/>
+  <child link="camera_rotate_servo_1"/>
+  <axis xyz="0.0 0.0 1.0"/>
+</joint>
+<joint name="joint_cam_tilt" type="continuous">
+  <origin xyz="-0.015 0.0 0.01" rpy="0 0 0"/>
+  <parent link="camera_rotate_servo_1"/>
+  <child link="camera_tilt_servo_1"/>
+  <axis xyz="0.0 1.0 0.0"/>
+</joint>
 </robot>

Commit message: lidar

File: urdf/AutoCar.xacro (robot description, xacro)
@@ -6,7 +6,7 @@
 <link name="base_link">
   <inertial>
-    <origin xyz="-0.0008559347867336729 -1.0776657557532648e-16 0.032797715315650726" rpy="0 0 0"/>
-    <mass value="42.39998679844243"/>
-    <inertia ixx="0.138613" iyy="1.488522" izz="1.592956" ixy="-0.0" iyz="-0.0" ixz="-0.006017"/>
+    <origin xyz="0.006241047940893729 1.7542466020202997e-05 0.04792208933122006" rpy="0 0 0"/>
+    <mass value="51.74527306163868"/>
+    <inertia ixx="0.210744" iyy="1.719578" izz="1.775248" ixy="-0.00012" iyz="-9.1e-05" ixz="-0.04364"/>
   </inertial>
   <visual>
@@ -141,4 +141,24 @@
     <geometry>
       <mesh filename="file://$(find auto_car_description)/meshes/camera_tilt_servo_1.stl" scale="0.001 0.001 0.001"/>
+    </geometry>
+  </collision>
+</link>
+<link name="lidar_1">
+  <inertial>
+    <origin xyz="-1.4978991194625202e-07 -6.94672942983649e-08 0.018020517916249423" rpy="0 0 0"/>
+    <mass value="1.2797567850628393"/>
+    <inertia ixx="0.000591" iyy="0.000591" izz="0.000902" ixy="-0.0" iyz="0.0" ixz="0.0"/>
+  </inertial>
+  <visual>
+    <origin xyz="-0.138818 -0.000316 -0.176" rpy="0 0 0"/>
+    <geometry>
+      <mesh filename="file://$(find auto_car_description)/meshes/lidar_1.stl" scale="0.001 0.001 0.001"/>
+    </geometry>
+    <material name="silver"/>
+  </visual>
+  <collision>
+    <origin xyz="-0.138818 -0.000316 -0.176" rpy="0 0 0"/>
+    <geometry>
+      <mesh filename="file://$(find auto_car_description)/meshes/lidar_1.stl" scale="0.001 0.001 0.001"/>
     </geometry>
   </collision>
@@ -210,3 +230,9 @@
   <axis xyz="0.0 1.0 0.0"/>
 </joint>
+<joint name="joint_lidar" type="continuous">
+  <origin xyz="0.138818 0.000316 0.176" rpy="0 0 0"/>
+  <parent link="base_link"/>
+  <child link="lidar_1"/>
+  <axis xyz="0.0 0.0 1.0"/>
+</joint>
 </robot>

Commit message: imu

File: urdf/AutoCar.xacro (robot description, xacro)
@@ -194,4 +194,22 @@
   <limit effort="10" lower="-0.34" upper="0.34" velocity="100"/>
 </joint>
+<link name="imu_link">
+  <collision>
+    <origin xyz="0 0 0" rpy="0 0 0"/>
+    <geometry>
+      <box size="0.1 0.1 0.1"/>
+    </geometry>
+  </collision>
+  <inertial>
+    <mass value="1e-5" />
+    <origin xyz="0 0 0" rpy="0 0 0"/>
+    <inertia ixx="1e-6" ixy="0" ixz="0" iyy="1e-6" iyz="0" izz="1e-6" />
+  </inertial>
+</link>
+<joint name="imu_joint" type="fixed">
+  <origin xyz="-0.039 0 0.0859" rpy="0 0 0"/>
+  <parent link="base_link"/>
+  <child link="imu_link"/>
+</joint>
 <joint name="joint_front_left" type="continuous">
   <origin xyz="0 0 0" rpy="0 0 0"/>
